File: PCBs/Controller/ParkingInformationSupervisionSystem/ParkingInformationSupervisionSystem.kicad_sch (KiCad schematic)
At the start: 23 parts, among them J1 08B0-1X1T-03-F, J2 Conn_01x04_Pin, J3 Conn_01x06_Pin, Q1 IRLZ44N, Q2 IRLZ44N, U1 MCU-PIC18F67J60-I_PT_TQFP64_, U2 STM32F446RET6, U3 W5500

Commit message: Updated schematic to be more clear for Dr. Lichter
Parts:
- removed C4: 100n, Capacitor_THT:C_Disc_D10.5mm_W5.0mm_P5.00mm, symbol Device:C
- removed J3: Conn_01x06_Pin, Connector_PinSocket_2.54mm:PinSocket_1x06_P2.54mm_Vertical, symbol Connector:Conn_01x06_Pin
- removed U1: MCU-PIC18F67J60-I_PT_TQFP64_, MCU-PIC18F67J60-I_PT_TQFP64_:TQFP64-0.5-12X12MM, symbol MCU-PIC18F67J60-I_PT_TQFP64_:MCU-PIC18F67J60-I_PT_TQFP64_
- added J3: Conn_01x04_Pin, Connector_PinSocket_2.54mm:PinSocket_1x04_P2.54mm_Vertical, symbol Connector:Conn_01x04_Pin
Connections:
- net gLS1: now also J3.2 (Pin_2)
- net rLS1: now also J3.3 (Pin_3)
- new net 12V: J3.1 (Pin_1)
Other:
- note added: "CONNECTION BETWEEN JACK AND CHIP IS INTERNAL, NOT INCLUDING"
- note added: "ETHERNET MODULE WIZ850io"
- note added: "MICROCONTROLLER (USING DEV BOARD, BUT THESE ARE THE INTERNAL PINS)"
- note added: "NC"
- note added: "PLACEHOLDER FOR TESTING"
- note added: "STACK LIGHT 1"
- note added: "TO DRIVER"
- note added: "TO ETH SWITCH"
- note added: "TO ETHERNET MODULE"
- note added: "TO P.S."
- note added: "TO POWER SUPPLY"
- note added: "TO STACK LIGHT"
- note added: "TO STATUS LIGHT DRIVER"
- note added: "TO uC"
- note removed: "ICSP HEADER"
- moved on the sheet: C1, C2, C3, C5, D1, D2, J1, J2, Q1, Q2, R1, R2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
